Commit message: fsdf

File: rikuken_robot/urdf/hande_camera.urdf.xacro (robot description, xacro)
@@ -23,5 +23,5 @@
             <visual>
                 <geometry>
-                    <mesh filename="package://tf_publish/meshes/body.dae"/>
+                    <mesh filename="package://rikuken_robot/meshes/body.dae"/>
                 </geometry>
                 <!--origin xyz="0.086 0 0" rpy="0.0 ${pi/2} 0.0"/-->
@@ -30,5 +30,5 @@
                <!--origin xyz="0.086 0 0" rpy="0.0 ${pi/2} 0.0"/-->
                 <geometry>
-                    <mesh filename="package://tf_publish/meshes/body.dae"/>
+                    <mesh filename="package://rikuken_robot/meshes/body.dae"/>
                 </geometry>
             </collision>
@@ -54,5 +54,5 @@
             <visual>
                 <geometry>
-                    <mesh filename="package://tf_publish/meshes/finger_11.dae"/>
+                    <mesh filename="package://rikuken_robot/meshes/finger_11.dae"/>
                 </geometry>
                 <material name="gray" />
@@ -62,5 +62,5 @@
                 <!--origin rpy="${pi/2} ${-pi/2} ${pi}" xyz="0.086 0 0"/-->
                 <geometry>
-                    <mesh filename="package://tf_publish/meshes/finger_11.dae"/>
+                    <mesh filename="package://rikuken_robot/meshes/finger_11.dae"/>
                 </geometry>
             </collision>
@@ -160,5 +160,5 @@
             <visual>
                 <geometry>
-                    <mesh filename="package://tf_publish/meshes/finger_22.dae"/>
+                    <mesh filename="package://rikuken_robot/meshes/finger_22.dae"/>
                 </geometry>
                 <material name="gray" />
@@ -168,5 +168,5 @@
                 <!--origin rpy="${-pi/2} ${3*pi/2} 0.0" xyz="0.086 0.02 0.0"/-->
                 <geometry>
-                    <mesh filename="package://tf_publish/meshes/finger_22.dae"/>
+                    <mesh filename="package://rikuken_robot/meshes/finger_22.dae"/>
                 </geometry>
             </collision>

File: rikuken_robot/urdf/ur3e.urdf.xacro (robot description, xacro)
@@ -4,6 +4,6 @@
   Author: Felix Messmer
 -->
-  <xacro:include filename="$(find tf_publish)/urdf/ur3e.transmission.xacro" />
-  <xacro:include filename="$(find tf_publish)/urdf/ur3e.gazebo.xacro" />
+  <xacro:include filename="$(find rikuken_robot)/urdf/ur3e.transmission.xacro" />
+  <xacro:include filename="$(find rikuken_robot)/urdf/ur3e.gazebo.xacro" />
   <xacro:macro name="cylinder_inertial" params="radius length mass *origin">
     <inertial>
@@ -55,5 +55,5 @@
         <origin xyz="0 0 0" rpy="0 0 ${base_correction}"/>
         <geometry>
-          <mesh filename="package://tf_publish/meshes/ur3e/visual/base.dae"/>
+          <mesh filename="package://rikuken_robot/meshes/ur3e/visual/base.dae"/>
         </geometry>
         <material name="LightGrey">
@@ -64,5 +64,5 @@
         <origin xyz="0 0 0" rpy="0 0 ${base_correction}"/>
         <geometry>
-          <mesh filename="package://tf_publish/meshes/ur3e/visual/base.dae"/>
+          <mesh filename="package://rikuken_robot/meshes/ur3e/visual/base.dae"/>
         </geometry>
       </collision>
@@ -94,5 +94,5 @@
         <origin xyz="0 0 0" rpy="0 0 ${pi}"/>
         <geometry>
-          <mesh filename="package://tf_publish/meshes/ur3e/visual/shoulder.dae"/>
+          <mesh filename="package://rikuken_robot/meshes/ur3e/visual/shoulder.dae"/>
         </geometry>
         <material name="LightGrey">
@@ -103,5 +103,5 @@
         <origin xyz="0 0 0" rpy="0 0 ${pi}"/>
         <geometry>
-          <mesh filename="package://tf_publish/meshes/ur3e/visual/shoulder.dae"/>
+          <mesh filename="package://rikuken_robot/meshes/ur3e/visual/shoulder.dae"/>
         </geometry>
       </collision>
@@ -133,5 +133,5 @@
         <origin xyz="0 0 ${shoulder_offset}" rpy="${pi/2} 0 ${-pi/2}"/>
         <geometry>
-          <mesh filename="package://tf_publish/meshes/ur3e/visual/upperarm.dae"/>
+          <mesh filename="package://rikuken_robot/meshes/ur3e/visual/upperarm.dae"/>
         </geometry>
         <material name="LightGrey">
@@ -142,5 +142,5 @@
         <origin xyz="0 0 ${shoulder_offset}" rpy="${pi/2} 0 ${-pi/2}"/>
         <geometry>
-          <mesh filename="package://tf_publish/meshes/ur3e/visual/upperarm.dae"/>
+          <mesh filename="package://rikuken_robot/meshes/ur3e/visual/upperarm.dae"/>
         </geometry>
       </collision>
@@ -172,5 +172,5 @@
         <origin xyz="0 0 ${elbow_offset}" rpy="${pi/2} 0 ${-pi/2}"/>
         <geometry>
-          <mesh filename="package://tf_publish/meshes/ur3e/visual/forearm.dae"/>
+          <mesh filename="package://rikuken_robot/meshes/ur3e/visual/forearm.dae"/>
         </geometry>
         <material name="LightGrey">
@@ -181,5 +181,5 @@
         <origin xyz="0 0 ${elbow_offset}" rpy="${pi/2} 0 ${-pi/2}"/>
         <geometry>
-          <mesh filename="package://tf_publish/meshes/ur3e/visual/forearm.dae"/>
+          <mesh filename="package://rikuken_robot/meshes/ur3e/visual/forearm.dae"/>
         </geometry>
       </collision>
@@ -211,5 +211,5 @@
         <origin xyz="0 0 -0.104" rpy="${pi/2} 0 0"/>
         <geometry>
-          <mesh filename="package://tf_publish/meshes/ur3e/visual/wrist1.dae"/>
+          <mesh filename="package://rikuken_robot/meshes/ur3e/visual/wrist1.dae"/>
         </geometry>
         <material name="LightGrey">
@@ -220,5 +220,5 @@
         <origin xyz="0 0 -0.104" rpy="${pi/2} 0 0"/>
         <geometry>
-          <mesh filename="package://tf_publish/meshes/ur3e/visual/wrist1.dae"/>
+          <mesh filename="package://rikuken_robot/meshes/ur3e/visual/wrist1.dae"/>
         </geometry>
       </collision>
@@ -250,5 +250,5 @@
         <origin xyz="0 0 -0.08535" rpy="0 0 0"/>
         <geometry>
-          <mesh filename="package://tf_publish/meshes/ur3e/visual/wrist2.dae"/>
+          <mesh filename="package://rikuken_robot/meshes/ur3e/visual/wrist2.dae"/>
         </geometry>
         <material name="LightGrey">
@@ -259,5 +259,5 @@
         <origin xyz="0 0 -0.08535" rpy="0 0 0"/>
         <geometry>
-          <mesh filename="package://tf_publish/meshes/ur3e/visual/wrist2.dae"/>
+          <mesh filename="package://rikuken_robot/meshes/ur3e/visual/wrist2.dae"/>
         </geometry>
       </collision>
@@ -289,5 +289,5 @@
         <origin xyz="0 0 -0.0921" rpy="${pi/2} 0 0"/>
         <geometry>
-          <mesh filename="package://tf_publish/meshes/ur3e/visual/wrist3.dae"/>
+          <mesh filename="package://rikuken_robot/meshes/ur3e/visual/wrist3.dae"/>
         </geometry>
         <material name="LightGrey">
@@ -298,5 +298,5 @@
         <origin xyz="0 0 -0.0921" rpy="${pi/2} 0 0"/>
         <geometry>
-          <mesh filename="package://tf_publish/meshes/ur3e/visual/wrist3.dae"/>
+          <mesh filename="package://rikuken_robot/meshes/ur3e/visual/wrist3.dae"/>
         </geometry>
       </collision>

File: rikuken_robot/urdf/ur3e_hand_E_camera.urdf.xacro (robot description, xacro)
@@ -2,6 +2,6 @@
 <robot xmlns:xacro="http://www.ros.org/wiki/xacro" name="ur3e_gripper">
   <!--xacro:include filename="$(find ur5_description)/urdf/ur5_joint_limited_robot.urdf.xacro" /-->
-  <xacro:include filename="$(find tf_publish)/urdf/ur3e_joint_limited_robot.urdf.xacro" />
-  <xacro:include filename="$(find tf_publish)/urdf/hande_camera.urdf.xacro" />
+  <xacro:include filename="$(find rikuken_robot)/urdf/ur3e_joint_limited_robot.urdf.xacro" />
+  <xacro:include filename="$(find rikuken_robot)/urdf/hande_camera.urdf.xacro" />
   <!-- Robotiq Coupler -->
   <!--  + Height added by the coupler: 8mm -->
@@ -10,5 +10,5 @@
     <visual>
       <geometry>
-        <mesh filename="package://tf_publish/meshes/robotiq_85_coupler.stl" />
+        <mesh filename="package://rikuken_robot/meshes/robotiq_85_coupler.stl" />
       </geometry>
       <material name="flat_black"/>
@@ -16,5 +16,5 @@
     <collision>
       <geometry>
-        <mesh filename="package://tf_publish/meshes/robotiq_85_coupler.stl" />
+        <mesh filename="package://rikuken_robot/meshes/robotiq_85_coupler.stl" />
       </geometry>
     </collision>

File: rikuken_robot/urdf/ur3e_joint_limited_robot.urdf.xacro (robot description, xacro)
@@ -3,9 +3,9 @@
   <xacro:arg name="transmission_hw_interface" default="hardware_interface/PositionJointInterface"/>
   <!-- common stuff -->
-  <xacro:include filename="$(find tf_publish)/urdf/ur3e_common.gazebo.xacro" />
+  <xacro:include filename="$(find rikuken_robot)/urdf/ur3e_common.gazebo.xacro" />
   <!-- ur3e -->
-  <xacro:include filename="$(find tf_publish)/urdf/ur3e.urdf.xacro" />
+  <xacro:include filename="$(find rikuken_robot)/urdf/ur3e.urdf.xacro" />
   <!-- arm -->
-  <xacro:arg name="kinematics_config" default="$(find tf_publish)/config/ur3e_default.yaml"/>
+  <xacro:arg name="kinematics_config" default="$(find rikuken_robot)/config/ur3e_default.yaml"/>
   <xacro:ur3e_robot prefix="" joint_limited="true"
     shoulder_pan_lower_limit="${-pi}" shoulder_pan_upper_limit="${pi}"
@@ -22,5 +22,6 @@
     <parent link="world" />
     <child link = "base_link" />
-    <origin xyz="-0.5 0.0 1.03" rpy="0.0 0.0 0.0" />
+    <!-- <origin xyz="-0.5 0.0 1.03" rpy="0.0 0.0 0.0" /> -->
+    <origin xyz="0 0 0" rpy="0.0 0.0 0.0" />
   </joint>
 </robot>
